File: analogkeyboard.kicad_pcb (KiCad board)
At the start: 2 copper layers, 77.5 x 35.6 mm, 50 parts, among them J1 AtinyCon

Commit message: Add files via upload
Parts:
- added ESPACE: SW_Push_45deg, stm32china:SW_SPST_B3U-1000P, F.Cu at (151.1, 109.2)
- added ESPACE: SW_Push_45deg, stm32china:SW_SPST_B3U-1000P, F.Cu at (158.8, 109.2)
- moved ESPACE 3.78 mm to (166.4, 109.2)
Routing:
- net Net-(D1-Pad1): track 55.4 -> 62.1 mm
